File: kicad/output.kicad_sch (KiCad schematic)
At the start: 6 parts, among them J10 Conn_01x03, J3 AudioJack3

Commit message: fix mixers in filter and compressor, update pcb
Parts:
- RV16, RV17: value 100K -> A100K
Connections:
- net GND: now also RV16.1, RV17.1; no longer RV16.3, RV17.3
- net at C19.2: now also RV17.3; no longer RV17.1
- net at C18.2: now also RV16.3; no longer RV16.1
Other:
- moved on the sheet: RV16, RV17
Changed lines of the file:
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@@
 	(symbol
 		(lib_id "Device:R_Potentiometer")
-		(at 119.38 97.79 90)
+		(at 119.38 97.79 270)
+		(mirror x)
 		(unit 1)
 		(exclude_from_sim no)
@@
 		(on_board yes)
 		(dnp no)
-		(fields_autoplaced yes)
 		(property "Reference" "RV17"
 			(at 119.38 101.6 90)
@@
 			)
 		)
-		(property "Value" "100K"
+		(property "Value" "A100K"
 			(at 119.38 104.14 90)
 			(effects
@@
 	(symbol
 		(lib_id "Device:R_Potentiometer")
-		(at 119.38 78.74 90)
+		(at 119.38 78.74 270)
+		(mirror x)
 		(unit 1)
 		(exclude_from_sim no)
@@
 		(on_board yes)
 		(dnp no)
-		(fields_autoplaced yes)
 		(property "Reference" "RV16"
 			(at 119.38 82.55 90)
@@
 			)
 		)
-		(property "Value" "100K"
+		(property "Value" "A100K"
 			(at 119.38 85.09 90)
 			(effects

Commit message: mark components as DNP, add LCSC part numbers
Parts:
- J10, J3, RV16, RV17: now not fitted
Changed lines of the file:
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@@
 		(in_bom yes)
 		(on_board yes)
-		(dnp no)
+		(dnp yes)
 		(fields_autoplaced yes)
 		(property "Reference" "J10"
@@
 		)
 		(property "Description" "Generic connector, single row, 01x03, script generated (kicad-library-utils/schlib/autogen/connector/)"
+			(at 74.93 57.15 0)
+			(effects
+				(font
+					(size 1.27 1.27)
+				)
+				(hide yes)
+			)
+		)
+		(property "LCSC Part" ""
 			(at 74.93 57.15 0)
 			(effects
@@
 		)
 		(property "Description" "Unpolarized capacitor, small symbol"
+			(at 105.41 97.79 0)
+			(effects
+				(font
+					(size 1.27 1.27)
+				)
+				(hide yes)
+			)
+		)
+		(property "LCSC Part" ""
 			(at 105.41 97.79 0)
 			(effects
@@
 		(in_bom yes)
 		(on_board yes)
-		(dnp no)
+		(dnp yes)
 		(property "Reference" "RV17"
 			(at 119.38 101.6 90)
@@
 		)
 		(property "Description" "Potentiometer"
+			(at 119.38 97.79 0)
+			(effects
+				(font
+					(size 1.27 1.27)
+				)
+				(hide yes)
+			)
+		)
+		(property "LCSC Part" ""
 			(at 119.38 97.79 0)
 			(effects
@@
 		(in_bom yes)
 		(on_board yes)
-		(dnp no)
+		(dnp yes)
 		(property "Reference" "RV16"
 			(at 119.38 82.55 90)
@@
 		)
 		(property "Description" "Potentiometer"
+			(at 119.38 78.74 0)
+			(effects
+				(font
+					(size 1.27 1.27)
+				)
+				(hide yes)
+			)
+		)
+		(property "LCSC Part" ""
 			(at 119.38 78.74 0)
 			(effects
@@
 			)
 		)
+		(property "LCSC Part" ""
+			(at 105.41 78.74 0)
+			(effects
+				(font
+					(size 1.27 1.27)
+				)
+				(hide yes)
+			)
+		)
 		(pin "1"
 		)
@@
 		(in_bom yes)
 		(on_board yes)
-		(dnp no)
+		(dnp yes)
 		(fields_autoplaced yes)
 		(property "Reference" "J3"
@@
 			(at 158.75 86.36 0)
 			(effects
+				(font
+					(size 1.27 1.27)
+				)
+				(hide yes)
+			)
+		)
+		(property "LCSC Part" ""
+			(at 158.75 86.36 0)
+			(effects

Commit message: add local changes
Other:
- note removed: "tbd: log potis?"
Changed lines of the file:
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@@
-		)
-	)
-	(text "tbd: log potis?\n"
-		(exclude_from_sim no)
-		(at 129.032 115.062 0)
-		(effects
-			(font
-				(size 1.27 1.27)
-			)
 		)
 	)
